Commit message: fix split gazebo config

File: src/machine/robot_description/urdf/robot.gazebo.xacro (robot description, xacro)
@@ -1,4 +1,4 @@
-<?xml version="1.0" encoding="utf-8"?>
-<robot name="robot" xmlns:xacro="http://www.ros.org/wiki/xacro" >
+<?xml version="1.0"?>
+<robot xmlns:xacro="http://www.ros.org/wiki/xacro" >
   <gazebo>
     <plugin name="differential_drive_controller" filename="libgazebo_ros_diff_drive.so">

File: src/machine/robot_description/urdf/robot.xacro (robot description, xacro)
@@ -1,388 +1,388 @@
 <?xml version="1.0" encoding="utf-8"?>
 <robot name="robot" xmlns:xacro="http://www.ros.org/wiki/xacro">
-    <!-- Gazebo configuration -->
-    <xacro:include filename="$(find robot_description)/urdf/robot.gazebo.xacro" />
-    <!-- Robot configuration -->
-    <link name="base_footprint"/>
-    <joint name="base_joint" type="fixed">
-      <origin xyz="0 0 0.05" rpy="0 0 0" />
-      <parent link="base_footprint"/>
-      <child link="base_link" />
-    </joint>
-    <link name="base_link">
-      <visual>
-        <geometry>
-          <mesh filename="package://robot_description/meshes/base.dae"/>
-        </geometry>
-        <origin xyz="-0.52 -0.4 0.43" rpy="0 0 0"/>
-      </visual>
-      <collision>
-        <geometry>
-          <mesh filename="package://robot_description/meshes/base.dae"/>
-        </geometry>
-        <origin xyz="-0.52 -0.4 0.43" rpy="0 0 0"/>
-      </collision>
-      <inertial>
-        <origin xyz="0.0 0 0."/>
-        <mass value="0.5"/>
-        <inertia ixx="0.01" ixy="0.0" ixz="0.0"
-                 iyy="0.01" iyz="0.0"
-                 izz="0.03" />
-      </inertial>
-    </link>
-    <joint name="second_level_joint" type="fixed">
-      <origin xyz="0 0 0.68" rpy="0 0 0" />
-      <parent link="base_link"/>
-      <child link="base_second_link" />
-    </joint>
-    <link name="base_second_link">
-      <visual>
-        <geometry>
-          <mesh filename="package://robot_description/meshes/base.dae"/>
-        </geometry>
-        <origin xyz="-0.52 -0.4 0.0" rpy="0 0 0"/>
-      </visual>
-      <collision>
-        <geometry>
-          <mesh filename="package://robot_description/meshes/base.dae"/>
-        </geometry>
-        <origin xyz="-0.52 -0.4 0.0" rpy="0 0 0"/>
-      </collision>
-      <!--inertial>
-        <origin xyz="0.01 0 0.7"/>
-        <mass value="1.0"/>
-        <inertia ixx="0.01" ixy="0.0" ixz="0.0"
-                 iyy="0.01" iyz="0.0"
-                 izz="0.03" />
-      </inertial-->
-    </link>
-    <joint name="mcu_joint" type="fixed">
-      <origin xyz="0.02 0.12 0.73" rpy="0 0 0" />
-      <parent link="base_link"/>
-      <child link="mcu_link" />
-    </joint>
-    <link name="mcu_link">
-      <visual>
-        <geometry>
-          <mesh filename="package://robot_description/meshes/rasp.dae" scale="0.14 0.14 0.14"/>
-        </geometry>
-        <origin xyz="0.9 -1.25 0" rpy="0 0 1.57"/>
-      </visual>
-      <collision>
-        <geometry>
-          <mesh filename="package://robot_description/meshes/rasp.dae" scale="0.14 0.14 0.14"/>
-        </geometry>
-        <origin xyz="0.9 -1.25 0" rpy="0 0 1.57"/>
-      </collision>
-      <!-- inertial>
-        <origin xyz="0.01 0 0"/>
-        <mass value="1.0"/>
-        <inertia ixx="0.019995" ixy="0.0" ixz="0.0"
-                 iyy="0.019995" iyz="0.0"
-                 izz="0.03675" />
-      </inertial-->
-    </link>
-   <joint name="mcu_joint_1" type="fixed">
-      <origin xyz="0.02 0.12 0.83" rpy="0 0 0" />
-      <parent link="base_link"/>
-      <child link="mcu_link_1" />
-    </joint>
-    <link name="mcu_link_1">
-      <visual>
-        <geometry>
-          <mesh filename="package://robot_description/meshes/rasp.dae" scale="0.14 0.14 0.14"/>
-        </geometry>
-        <origin xyz="0.9 -1.25 0" rpy="0 0 1.57"/>
-      </visual>
-      <collision>
-        <geometry>
-          <mesh filename="package://robot_description/meshes/rasp.dae" scale="0.14 0.14 0.14"/>
-        </geometry>
-        <origin xyz="0.9 -1.25 0" rpy="0 0 1.57"/>
-      </collision>
-      <!-- inertial>
-        <origin xyz="0.01 0 0"/>
-        <mass value="1.0"/>
-        <inertia ixx="0.019995" ixy="0.0" ixz="0.0"
-                 iyy="0.019995" iyz="0.0"
-                 izz="0.03675" />
-      </inertial-->
-    </link>
-   <joint name="stand_mcu1_joint" type="fixed">
-      <origin xyz="0.02 0.25 0.78" rpy="0 0 1.57" />
-      <parent link="base_link"/>
-      <child link="stand_mcu1_link" />
-    </joint>
-    <link name="stand_mcu1_link">
-      <visual>
-        <geometry>
-         <cylinder length="0.1" radius="0.01"/>
-        </geometry>
-        <origin rpy="0.0 0 0" xyz="0 0 0.0"/>
-      </visual>
-      <collision>
-        <geometry>
-         <cylinder length="0.1" radius="0.01"/>
-        </geometry>
-        <origin rpy="0.0 0 0" xyz="0 0 0.0"/>
-      </collision>
-    </link>
-   <joint name="stand_mcu2_joint" type="fixed">
-      <origin xyz="0.02 -0.1125 0.78" rpy="0 0 1.57" />
-      <parent link="base_link"/>
-      <child link="stand_mcu2_link" />
-    </joint>
-    <link name="stand_mcu2_link">
-      <visual>
-        <geometry>
-         <cylinder length="0.1" radius="0.01"/>
-        </geometry>
-        <origin rpy="0.0 0 0" xyz="0 0 0.0"/>
-      </visual>
-      <collision>
-        <geometry>
-         <cylinder length="0.1" radius="0.01"/>
-        </geometry>
-        <origin rpy="0.0 0 0" xyz="0 0 0.0"/>
-      </collision>
-    </link>
-   <joint name="stand_mcu3_joint" type="fixed">
-      <origin xyz="0.25 0.25 0.78" rpy="0 0 1.57" />
-      <parent link="base_link"/>
-      <child link="stand_mcu3_link" />
-    </joint>
-    <link name="stand_mcu3_link">
-      <visual>
-        <geometry>
-         <cylinder length="0.1" radius="0.01"/>
-        </geometry>
-        <origin rpy="0.0 0 0" xyz="0 0 0.0"/>
-      </visual>
-      <collision>
-        <geometry>
-         <cylinder length="0.1" radius="0.01"/>
-        </geometry>
-        <origin rpy="0.0 0 0" xyz="0 0 0.0"/>
-      </collision>
-    </link>
-   <joint name="stand_mcu4_joint" type="fixed">
-      <origin xyz="0.25 -0.1125 0.78" rpy="0 0 1.57" />
-      <parent link="base_link"/>
-      <child link="stand_mcu4_link" />
-    </joint>
-    <link name="stand_mcu4_link">
-      <visual>
-        <geometry>
-         <cylinder length="0.1" radius="0.01"/>
-        </geometry>
-        <origin rpy="0.0 0 0" xyz="0 0 0.0"/>
-      </visual>
-      <collision>
-        <geometry>
-         <cylinder length="0.1" radius="0.01"/>
-        </geometry>
-        <origin rpy="0.0 0 0" xyz="0 0 0.0"/>
-      </collision>
-    </link>
-    <joint name="batery_joint" type="fixed">
-      <origin xyz="1.2 0.2 0.43" rpy="0 0 1.57" />
-      <parent link="base_link"/>
-      <child link="batery_link" />
-    </joint>
-    <link name="batery_link">
-      <visual>
-        <geometry>
-          <mesh filename="package://robot_description/meshes/battery.dae" scale="13.0 6.0 6.0"/>
-        </geometry>
-        <origin xyz="0 4.5 0.05" rpy="1.57 0 1.57"/>
-      </visual>
-      <collision>
-        <geometry>
-          <mesh filename="package://robot_description/meshes/battery.dae" scale="13.0 6.0 6.0"/>
-        </geometry>
-        <origin xyz="0 4.5 0.05" rpy="1.57 0 1.57"/>
-      </collision>
-      <!-- inertial>
-        <origin xyz="0.01 0 0"/>
-        <mass value="1.0"/>
-        <inertia ixx="0.01" ixy="0.0" ixz="0.0"
-                 iyy="0.01" iyz="0.0"
-                 izz="0.03" />
-      </inertial-->
-    </link>
-   <joint name="stand_1_joint" type="fixed">
-      <origin xyz="0.5 0.4125 0.58" rpy="0 0 1.57" />
-      <parent link="base_link"/>
-      <child link="stand_1_link" />
-    </joint>
-    <link name="stand_1_link">
-      <visual>
-        <geometry>
-         <cylinder length="0.20" radius="0.03"/>
-        </geometry>
-        <origin rpy="0.0 0 0" xyz="0 0 0.0"/>
-      </visual>
-      <collision>
-        <geometry>
-         <cylinder length="0.20" radius="0.03"/>
-        </geometry>
-        <origin rpy="0.0 0 0" xyz="0 0 0.0"/>
-      </collision>
-      <!--inertial>
-        <origin xyz="0.0 0 0"/>
-        <mass value="1.0"/>
-        <inertia ixx="0.019995" ixy="0.0" ixz="0.0"
-                 iyy="0.019995" iyz="0.0"
-                 izz="0.03675" />
-      </inertial-->
-    </link>
-   <joint name="stand_2_joint" type="fixed">
-      <origin xyz="0.5 -0.2625 0.58" rpy="0 0 1.57" />
-      <parent link="base_link"/>
-      <child link="stand_2_link" />
-    </joint>
-    <link name="stand_2_link">
-      <visual>
-        <geometry>
-         <cylinder length="0.20" radius="0.03"/>
-        </geometry>
-        <origin rpy="0.0 0 0" xyz="0 0 0.0"/>
-      </visual>
-      <collision>
-        <geometry>
-         <cylinder length="0.20" radius="0.03"/>
-        </geometry>
-        <origin rpy="0.0 0 0" xyz="0 0 0.0"/>
-      </collision>
-      <!--inertial>
-        <origin xyz="0.0 0 0"/>
-        <mass value="1.0"/>
-        <inertia ixx="0.019995" ixy="0.0" ixz="0.0"
-                 iyy="0.019995" iyz="0.0"
-                 izz="0.03675" />
-      </inertial-->
-    </link>
-    <joint name="wheel_left_joint" type="continuous">
-      <parent link="base_link"/>
-      <child link="wheel_left_link"/>
-      <origin xyz="0.15 0.4125 0.30" rpy="-1.57 0 0"/>
-      <axis xyz="0 0 1"/>
-    </joint>
-    <link name="wheel_left_link">
-      <collision>
-        <geometry>
-         <cylinder length="0.20" radius="0.23"/>
-        </geometry>
-        <origin rpy="0.0 0.0 0" xyz="0 0 0.1"/>
-      </collision>
-      <visual name="visual">
-        <geometry>
-          <!-- cylinder length="0.0206" radius="0.0550"/-->
-          <!--cylinder length="0.20" radius="0.26"/-->
-          <mesh filename="package://robot_description/meshes/wheel.dae" scale="8.0 8.0 8.0"/>
-        </geometry>
-        <origin rpy="0.0 0 0" xyz="0 0 0"/>
-      </visual>
-      <inertial>
-        <mass value="0.4" />
-        <origin xyz="0 0 0" />
-        <inertia ixx="0.001" ixy="0.0" ixz="0.0"
-                 iyy="0.001" iyz="0.0"
-                 izz="0.001" />
-      </inertial>
-    </link>
-    <joint name="wheel_right_joint" type="continuous">
-      <parent link="base_link"/>
-      <child link="wheel_right_link"/>
-      <origin xyz="0.15 -0.5625 0.30" rpy="-1.57 0 0"/>
-      <axis xyz="0 0 1"/>
-    </joint>
-    <link name="wheel_right_link">
-      <collision>
-        <geometry>
-         <cylinder length="0.20" radius="0.23"/>
-        </geometry>
-        <origin rpy="0.0 0 0" xyz="0 0 0.195"/>
-      </collision>
-      <visual name="visual">
-        <geometry>
-	  <!--cylinder length="0.20" radius="0.26"/-->
-          <mesh filename="package://robot_description/meshes/wheel.dae" scale="8.0 8.0 8.0"/>
-        </geometry>
-        <origin rpy="0.0 0 0" xyz="0 0 0"/>
-      </visual>
-      <inertial>
-        <mass value="0.4" />
-        <origin xyz="0 0.0 0.3" />
-        <inertia ixx="0.001" ixy="0.0" ixz="0.0"
-                 iyy="0.001" iyz="0.0"
-                 izz="0.001" />
-      </inertial>
-    </link>
-    <joint name="caster_back_joint" type="fixed">
-      <parent link="base_link"/>
-      <child link="caster_back_link"/>
-      <origin xyz="-0.4 0.1 0.26" rpy="0 0 0"/>
-    </joint>
-    <link name="caster_back_link">
-      <collision>
-        <geometry>
-          <!-- cylinder length="0.05" radius="0.19"/-->
-          <sphere radius="0.19"/>
-        </geometry>
-        <origin rpy="0 0 0" xyz="0 0 0"/>
-      </collision>
-      <visual>
-        <geometry>
-          <!--cylinder length="0.05" radius="0.19"/-->
-          <sphere radius="0.19"/>
-        </geometry>
-        <origin rpy="0 0 0" xyz="0 0 0"/>
-      </visual>
-      <inertial>
-        <mass value="0.1" />
-        <origin xyz="0 0 0" />
-        <inertia ixx="0.001023539" ixy="0.0" ixz="0.0"
-                 iyy="0.001023539" iyz="0.0"
-                 izz="0.001023539" />
-      </inertial>
-    </link>
-   <joint name="stand_3_joint" type="fixed">
-      <origin xyz="-0.4 0.4125 0.58" rpy="0 0 1.57" />
-      <parent link="base_link"/>
-      <child link="stand_3_link" />
-    </joint>
-    <link name="stand_3_link">
-      <visual>
-        <geometry>
-         <cylinder length="0.20" radius="0.03"/>
-        </geometry>
-        <origin rpy="0.0 0 0" xyz="0 0 0.0"/>
-      </visual>
-      <collision>
-        <geometry>
-         <cylinder length="0.20" radius="0.03"/>
-        </geometry>
-        <origin rpy="0.0 0 0" xyz="0 0 0.0"/>
-      </collision>
-    </link>
-   <joint name="stand_4_joint" type="fixed">
-      <origin xyz="-0.4 -0.2625 0.58" rpy="0 0 1.57" />
-      <parent link="base_link"/>
-      <child link="stand_4_link" />
-    </joint>
-    <link name="stand_4_link">
-      <visual>
-        <geometry>
-         <cylinder length="0.20" radius="0.03"/>
-        </geometry>
-        <origin rpy="0.0 0 0" xyz="0 0 0.0"/>
-      </visual>
-      <collision>
-        <geometry>
-         <cylinder length="0.20" radius="0.03"/>
-        </geometry>
-        <origin rpy="0.0 0 0" xyz="0 0 0.0"/>
-      </collision>
-    </link>
+  <!-- Gazebo configuration -->
+  <xacro:include filename="$(find robot_description)/urdf/robot.gazebo.xacro" />
+  <!-- Robot configuration -->
+  <link name="base_footprint"/>
+  <joint name="base_joint" type="fixed">
+    <origin xyz="0 0 0.05" rpy="0 0 0" />
+    <parent link="base_footprint"/>
+    <child link="base_link" />
+  </joint>
+  <link name="base_link">
+    <visual>
+      <geometry>
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
Commit message: added camera and imu gazebo plugin

File: src/machine/robot_description/urdf/robot.gazebo.xacro (robot description, xacro)
@@ -1,4 +1,5 @@
 <?xml version="1.0"?>
 <robot xmlns:xacro="http://www.ros.org/wiki/xacro" >
+  <!-- Fake Control Plugin -->
   <gazebo>
     <plugin name="differential_drive_controller" filename="libgazebo_ros_diff_drive.so">
@@ -21,3 +22,82 @@
     </plugin>
   </gazebo>
+  <!-- Camera Plugin -->
+  <gazebo reference="camera_link">
+    <sensor type="camera" name="camera1">
+      <update_rate>30.0</update_rate>
+      <camera name="head">
+        <horizontal_fov>1.04</horizontal_fov>
+        <image>
+          <width>320</width>
+          <height>240</height>
+          <format>R8G8B8</format>
+        </image>
+        <clip>
+          <near>0.1</near>
+          <far>50</far>
+        </clip>
+      </camera>
+      <plugin name="camera_controller" filename="libgazebo_ros_camera.so">
+        <alwaysOn>true</alwaysOn>
+        <updateRate>0</updateRate>
+        <cameraName>camera1</cameraName>
+        <imageTopicName>image_raw</imageTopicName>
+        <cameraInfoTopicName>camera_info</cameraInfoTopicName>
+        <frameName>camera</frameName>
+        <hackBaseline>0.07</hackBaseline>
+        <distortionK1>0.0</distortionK1>
+        <distortionK2>0.0</distortionK2>
+        <distortionK3>0.0</distortionK3>
+        <distortionT1>0.0</distortionT1>
+        <distortionT2>0.0</distortionT2>
+      </plugin>
+    </sensor>
+  </gazebo>
+  <!-- IMU Plugin -->
+  <gazebo>
+    <plugin name="gazebo_ros_imu_controller" filename="libgazebo_ros_imu.so">
+      <!-- <robotNamespace></robotNamespace> -->
+      <topicName>imu/data</topicName>
+      <serviceName>imu/service</serviceName>
+      <bodyName>base_link</bodyName>
+      <gaussianNoise>0</gaussianNoise>
+      <rpyOffsets>0 0 0</rpyOffsets>
+      <updateRate>30.0</updateRate>
+      <alwaysOn>true</alwaysOn>
+      <gaussianNoise>0</gaussianNoise>
+    </plugin>
+  </gazebo>
+  <gazebo reference="wheel_left_link">
+    <mu1>1.0</mu1>
+    <mu2>1.0</mu2>
+    <kp>1000000.0</kp>
+    <kd>100.0</kd>
+    <minDepth>0.001</minDepth>
+    <maxVel>1.0</maxVel>
+  </gazebo>
+  <gazebo reference="wheel_right_link">
+    <mu1>1.0</mu1>
+    <mu2>1.0</mu2>
+    <kp>1000000.0</kp>
+    <kd>100.0</kd>
+    <minDepth>0.001</minDepth>
+    <maxVel>1.0</maxVel>
+  </gazebo>
+  <gazebo reference="base_link">
+    <material>Gazebo/Blue</material>
+    <mu1>0.3</mu1>
+    <mu2>0.3</mu2>
+    <sensor type="contact" name="bumpers">
+      <always_on>1</always_on>
+      <update_rate>50.0</update_rate>
+      <visualize>true</visualize>
+      <contact>
+        <collision>base_footprint_collision_base_link</collision>
+      </contact>
+    </sensor>
+  </gazebo>
+  <gazebo reference="camera_link">
+    <mu1>0.2</mu1>
+    <mu2>0.2</mu2>
+  </gazebo>
 </robot>

File: src/machine/robot_description/urdf/robot.xacro (robot description, xacro)
@@ -1,7 +1,7 @@
 <?xml version="1.0" encoding="utf-8"?>
 <robot name="robot" xmlns:xacro="http://www.ros.org/wiki/xacro">
-  <!-- Gazebo configuration -->
+<!-- Gazebo configuration -->
   <xacro:include filename="$(find robot_description)/urdf/robot.gazebo.xacro" />
-  <!-- Robot configuration -->
+<!-- Robot configuration -->
   <link name="base_footprint"/>
   <joint name="base_joint" type="fixed">
@@ -386,3 +386,24 @@
     </collision>
   </link>
+  <!-- Robot Sensors -->
+  <!-- Camera -->
+  <joint name="camera_joint" type="fixed">
+    <origin xyz="0.49 -0.03 0.75" rpy="0 0.21 0" />
+    <parent link="base_link"/>
+    <child link="camera_link" />
+  </joint>
+  <link name="camera_link">
+    <visual>
+      <geometry>
+        <mesh filename="package://robot_description/meshes/camera.dae" scale="4.0 4.0 4.0"/>
+      </geometry>
+      <origin xyz="0.0 0 0" rpy="0 0 0"/>
+    </visual>
+    <collision>
+      <geometry>
+        <mesh filename="package://robot_description/meshes/camera.dae" scale="4.0 4.0 4.0"/>
+      </geometry>
+      <origin xyz="0.0 0 0" rpy="0 0 0"/>
+    </collision>
+  </link>
 </robot>
