Commit message: update arm

File: src/machine/robot_description/urdf/arm.xacro (robot description, xacro)
@@ -1,32 +1,25 @@
 <?xml version="1.0"?>
 <robot xmlns:xacro="http://www.ros.org/wiki/xacro">
-  <!-- Propiedades comunes para el brazo (puedes incluir common_properties.xacro si quieres) -->
-  <!-- <xacro:include filename="$(find robot_description)/urdf/common_properties.xacro" /> -->
-  <!-- Definición de materiales básicos para el brazo (si no usas common_properties) -->
-  <material name="arm_grey">
-    <color rgba="0.7 0.7 0.7 1"/>
-  </material>
-  <material name="arm_black">
-    <color rgba="0.1 0.1 0.1 1"/>
-  </material>
+  <!-- Incluir propiedades comunes para materiales (ya se incluye en robot.xacro, pero se añade para claridad) -->
+  <xacro:include filename="$(find robot_description)/urdf/common_properties.xacro" />
   <!-- Base del brazo (se conectará a la base del robot principal) -->
   <link name="arm_base_link">
     <visual>
       <geometry>
-        <box size="0.1 0.1 0.05"/>
+        <box size="0.15 0.15 0.03"/> <!-- Base más ancha y plana -->
       </geometry>
-      <material name="arm_grey"/>
+      <material name="grey"/> <!-- Usando material de common_properties -->
     </visual>
     <collision>
       <geometry>
-        <box size="0.1 0.1 0.05"/>
+        <box size="0.15 0.15 0.03"/>
       </geometry>
     </collision>
     <inertial>
       <origin xyz="0 0 0" rpy="0 0 0"/>
-      <mass value="0.5"/>
-      <inertia ixx="0.001" ixy="0.0" ixz="0.0"
-               iyy="0.001" iyz="0.0"
-               izz="0.001"/>
+      <mass value="0.7"/>
+      <inertia ixx="0.002" ixy="0.0" ixz="0.0"
+               iyy="0.002" iyz="0.0"
+               izz="0.002"/>
     </inertial>
   </link>
@@ -35,26 +28,28 @@
     <parent link="arm_base_link"/>
     <child link="shoulder_link"/>
-    <origin xyz="0 0 0.025" rpy="0 0 0"/> <!-- Encima de la base del brazo -->
+    <origin xyz="0 0 0.015" rpy="0 0 0"/> <!-- Posición encima de la base del brazo -->
     <axis xyz="0 0 1"/> <!-- Rotación alrededor del eje Z (horizontal) -->
-    <limit lower="-1.57" upper="1.57" effort="100" velocity="0.5"/>
+    <limit lower="-1.8" upper="1.8" effort="100" velocity="0.5"/>
   </joint>
   <link name="shoulder_link">
     <visual>
       <geometry>
-        <box size="0.05 0.05 0.2"/>
+        <cylinder radius="0.05" length="0.25"/> <!-- Cilindro para el segmento del brazo -->
       </geometry>
-      <material name="arm_black"/>
+      <origin xyz="0 0 0.125" rpy="0 0 0"/> <!-- Centrar el cilindro para que extienda hacia arriba -->
+      <material name="blue"/> <!-- Color diferente para el segmento -->
     </visual>
     <collision>
       <geometry>
-        <box size="0.05 0.05 0.2"/>
+        <cylinder radius="0.05" length="0.25"/>
       </geometry>
+      <origin xyz="0 0 0.125" rpy="0 0 0"/>
     </collision>
     <inertial>
-      <origin xyz="0 0 0.1" rpy="0 0 0"/>
-      <mass value="0.5"/>
-      <inertia ixx="0.001" ixy="0.0" ixz="0.0"
-               iyy="0.001" iyz="0.0"
-               izz="0.001"/>
+      <origin xyz="0 0 0.125" rpy="0 0 0"/>
+      <mass value="0.6"/>
+      <inertia ixx="0.0015" ixy="0.0" ixz="0.0"
+               iyy="0.0015" iyz="0.0"
+               izz="0.0015"/>
     </inertial>
   </link>
@@ -63,26 +58,28 @@
     <parent link="shoulder_link"/>
     <child link="elbow_link"/>
-    <origin xyz="0 0 0.2" rpy="0 0 0"/> <!-- En la parte superior del hombro -->
+    <origin xyz="0 0 0.25" rpy="0 0 0"/> <!-- En la parte superior del eslabón del hombro -->
     <axis xyz="0 1 0"/> <!-- Rotación alrededor del eje Y (vertical) -->
-    <limit lower="-1.57" upper="1.57" effort="100" velocity="0.5"/>
+    <limit lower="-1.8" upper="1.8" effort="100" velocity="0.5"/>
   </joint>
   <link name="elbow_link">
     <visual>
       <geometry>
-        <box size="0.04 0.04 0.15"/>
+        <cylinder radius="0.04" length="0.20"/> <!-- Cilindro más pequeño -->
       </geometry>
-      <material name="arm_grey"/>
+      <origin xyz="0 0 0.1" rpy="0 0 0"/>
+      <material name="grey"/>
     </visual>
     <collision>
       <geometry>
-        <box size="0.04 0.04 0.15"/>
+        <cylinder radius="0.04" length="0.20"/>
       </geometry>
+      <origin xyz="0 0 0.1" rpy="0 0 0"/>
     </collision>
     <inertial>
-      <origin xyz="0 0 0.075" rpy="0 0 0"/>
-      <mass value="0.3"/>
-      <inertia ixx="0.0005" ixy="0.0" ixz="0.0"
-               iyy="0.0005" iyz="0.0"
-               izz="0.0005"/>
+      <origin xyz="0 0 0.1" rpy="0 0 0"/>
+      <mass value="0.4"/>
+      <inertia ixx="0.0008" ixy="0.0" ixz="0.0"
+               iyy="0.0008" iyz="0.0"
+               izz="0.0008"/>
     </inertial>
   </link>
@@ -91,22 +88,50 @@
     <parent link="elbow_link"/>
     <child link="wrist_link"/>
-    <origin xyz="0 0 0.15" rpy="0 0 0"/> <!-- En la parte superior del codo -->
+    <origin xyz="0 0 0.2" rpy="0 0 0"/> <!-- En la parte superior del eslabón del codo -->
     <axis xyz="0 1 0"/> <!-- Rotación alrededor del eje Y (vertical) -->
-    <limit lower="-1.57" upper="1.57" effort="100" velocity="0.5"/>
+    <limit lower="-1.8" upper="1.8" effort="100" velocity="0.5"/>
   </joint>
   <link name="wrist_link">
     <visual>
       <geometry>
-        <box size="0.03 0.03 0.05"/>
+        <cylinder radius="0.03" length="0.08"/> <!-- Cilindro aún más pequeño -->
       </geometry>
-      <material name="arm_black"/>
+      <origin xyz="0 0 0.04" rpy="0 0 0"/>
+      <material name="blue"/>
     </visual>
     <collision>
       <geometry>
-        <box size="0.03 0.03 0.05"/>
+        <cylinder radius="0.03" length="0.08"/>
+      </geometry>
+      <origin xyz="0 0 0.04" rpy="0 0 0"/>
+    </collision>
+    <inertial>
+      <origin xyz="0 0 0.04" rpy="0 0 0"/>
+      <mass value="0.15"/>
+      <inertia ixx="0.0002" ixy="0.0" ixz="0.0"
+               iyy="0.0002" iyz="0.0"
+               izz="0.0002"/>
+    </inertial>
+  </link>
+  <!-- Efector final (puede ser un simple cubo o un gripper más complejo) -->
+  <joint name="end_effector_joint" type="fixed">
+    <parent link="wrist_link"/>
+    <child link="end_effector_link"/>
+    <origin xyz="0 0 0.08" rpy="0 0 0"/> <!-- Posición al final de la muñeca -->
+  </joint>
+  <link name="end_effector_link">
+    <visual>
+      <geometry>
+        <box size="0.06 0.06 0.03"/> <!-- Caja simple para el efector final -->
+      </geometry>
+      <material name="grey"/>
+    </visual>
+    <collision>
+      <geometry>
+        <box size="0.06 0.06 0.03"/>
       </geometry>
     </collision>
     <inertial>
-      <origin xyz="0 0 0.025" rpy="0 0 0"/>
+      <origin xyz="0 0 0" rpy="0 0 0"/>
       <mass value="0.1"/>
       <inertia ixx="0.0001" ixy="0.0" ixz="0.0"
@@ -115,30 +140,3 @@
     </inertial>
   </link>
-  <!-- Puedes agregar un efector final (gripper, herramienta, etc.) aquí si lo deseas -->
-  <!-- Ejemplo de un efector final fijo -->
-  <joint name="end_effector_joint" type="fixed">
-    <parent link="wrist_link"/>
-    <child link="end_effector_link"/>
-    <origin xyz="0 0 0.025" rpy="0 0 0"/>
-  </joint>
-  <link name="end_effector_link">
-    <visual>
-      <geometry>
-        <box size="0.05 0.05 0.02"/>
-      </geometry>
-      <material name="arm_grey"/>
-    </visual>
-    <collision>
-      <geometry>
-        <box size="0.05 0.05 0.02"/>
-      </geometry>
-    </collision>
-    <inertial>
-      <origin xyz="0 0 0" rpy="0 0 0"/>
-      <mass value="0.05"/>
-      <inertia ixx="0.00005" ixy="0.0" ixz="0.0"
-               iyy="0.00005" iyz="0.0"
-               izz="0.00005"/>
-    </inertial>
-  </link>
 </robot>

File: src/machine/robot_description/urdf/robot.xacro (robot description, xacro)
@@ -64,5 +64,5 @@
     <!-- Ajusta estos valores xyz/rpy para posicionar el brazo donde desees en la base_second_link -->
     <!-- Por ejemplo, para colocarlo en el centro de la base_second_link si esta es la superficie superior -->
-    <origin xyz="0.0 0.0 0.0" rpy="0 0 0"/>
+    <origin xyz="0.5 -0.15 0.05" rpy="0 0 0"/>
   </joint>
   <joint name="mcu_joint" type="fixed">
