Commit message: update basic robot_b

File: src/machine/robot_b_description/urdf/robot.xacro (robot description, xacro)
@@ -1,25 +1,11 @@
 <?xml version="1.0" encoding="utf-8"?>
 <robot name="four_wheel_robot" xmlns:xacro="http://www.ros.org/wiki/xacro">
-  <!-- Definiciones de Materiales para las Visualizaciones -->
-  <material name="white">
-      <color rgba="1 1 1 0.5"/>
-  </material>
-  <material name="red">
-      <color rgba="1 0 0 1"/>
-  </material>
-  <material name="blue">
-      <color rgba="0.2 0.2 1 1"/>
-  </material>
-  <material name="black">
-      <color rgba="0 0 0 1"/>
-  </material>
-  <material name="grey">
-      <color rgba="0.5 0.5 0.5 1"/>
-  </material>
+  <!-- Common properties - Materials -->
+  <xacro:include filename="$(find robot_b_description)/urdf/common_properties.xacro" />
   <!-- Link base_footprint (convención ROS para la base del robot) -->
   <link name="base_footprint"/>
   <!-- Joint que conecta base_footprint con base_link -->
   <joint name="base_joint" type="fixed">
-    <origin xyz="0 0 0.1" rpy="0 0 0" />
+    <origin xyz="0 0 0.2" rpy="0 0 0" />
     <parent link="base_footprint"/>
     <child link="base_link" />
@@ -48,10 +34,10 @@
   </link>
   <!-- Macro para definir una rueda, facilitando la creación de las cuatro -->
-  <xacro:macro name="wheel" params="prefix parent_link x_offset y_offset">
+  <xacro:macro name="wheel" params="prefix parent_link x_offset y_offset z_offset">
     <joint name="${prefix}_wheel_joint" type="continuous">
       <parent link="${parent_link}"/>
       <child link="${prefix}_wheel_link"/>
       <!-- rpy="-1.570795 0 0" rota la rueda para que el eje Z apunte hacia afuera (horizontal) -->
-      <origin xyz="${x_offset} ${y_offset} 0" rpy="-1.570795 0 0"/>
+      <origin xyz="${x_offset} ${y_offset} ${z_offset} " rpy="-1.570795 0 0"/>
       <axis xyz="0 0 1"/> <!-- El eje de rotación de la rueda es su propio eje Z local -->
     </joint>
@@ -80,20 +66,10 @@
   <!-- Instanciamos las cuatro ruedas usando la macro -->
   <!-- Rueda Delantera Izquierda -->
-  <xacro:wheel prefix="front_left" parent_link="base_link" x_offset="0.2" y_offset="0.225"/>
+  <xacro:wheel prefix="front_left" parent_link="base_link" x_offset="0.2" y_offset="0.225" z_offset="-0.1"/>
   <!-- Rueda Delantera Derecha -->
-  <xacro:wheel prefix="front_right" parent_link="base_link" x_offset="0.2" y_offset="-0.225"/>
+  <xacro:wheel prefix="front_right" parent_link="base_link" x_offset="0.2" y_offset="-0.225" z_offset="-0.1"/>
   <!-- Rueda Trasera Izquierda -->
-  <xacro:wheel prefix="back_left" parent_link="base_link" x_offset="-0.2" y_offset="0.225"/>
+  <xacro:wheel prefix="back_left" parent_link="base_link" x_offset="-0.2" y_offset="0.225" z_offset="-0.1"/>
   <!-- Rueda Trasera Derecha -->
-  <xacro:wheel prefix="back_right" parent_link="base_link" x_offset="-0.2" y_offset="-0.225"/>
-  <!--
-  Para la simulación en Gazebo:
-  Normalmente, se incluiría un archivo `robot.gazebo.xacro` (similar a como se hace en `robot_test/robot.xacro`)
-  para definir los plugins de Gazebo. Para un robot de cuatro ruedas, el plugin `libgazebo_ros_diff_drive.so`
-  (usado para robots diferenciales de dos ruedas) no sería directamente aplicable a menos que se agrupen
-  las ruedas (por ejemplo, las dos izquierdas como una sola unidad de control y las dos derechas como otra).
-  Si deseas que las cuatro ruedas sean impulsadas independientemente o con un control más complejo para 4WD,
-  necesitarías un plugin de Gazebo o un controlador ROS diferente, o configurar el `diff_drive` para
-  controlar dos "pares" de ruedas.
-  -->
+  <xacro:wheel prefix="back_right" parent_link="base_link" x_offset="-0.2" y_offset="-0.225" z_offset="-0.1"/>
 </robot>
