Commit message: split in package robot_a and robot_b

File: src/machine/robot_a_description/urdf/arm.xacro (robot description, xacro)
@@ -2,5 +2,5 @@
 <robot xmlns:xacro="http://www.ros.org/wiki/xacro">
   <!-- Incluir propiedades comunes para materiales (ya se incluye en robot.xacro, pero se añade para claridad) -->
-  <xacro:include filename="$(find robot_description)/urdf/common_properties.xacro" />
+  <xacro:include filename="$(find robot_a_description)/urdf/common_properties.xacro" />
   <!-- Base del brazo (se conectará a la base del robot principal) -->
   <link name="arm_base_link">

File: src/machine/robot_a_description/urdf/robot.xacro (robot description, xacro)
@@ -2,5 +2,5 @@
 <robot name="robot" xmlns:xacro="http://www.ros.org/wiki/xacro">
 <!-- Gazebo configuration -->
-  <xacro:include filename="$(find robot_description)/urdf/robot.gazebo.xacro" />
+  <xacro:include filename="$(find robot_a_description)/urdf/robot.gazebo.xacro" />
 <!-- Robot configuration -->
   <link name="base_footprint"/>
@@ -13,5 +13,5 @@
     <visual>
       <geometry>
-        <mesh filename="package://robot_description/meshes/base.dae"/>
+        <mesh filename="package://robot_a_description/meshes/base.dae"/>
       </geometry>
       <origin xyz="-0.52 -0.4 0.43" rpy="0 0 0"/>
@@ -19,5 +19,5 @@
     <collision>
       <geometry>
-        <mesh filename="package://robot_description/meshes/base.dae"/>
+        <mesh filename="package://robot_a_description/meshes/base.dae"/>
       </geometry>
       <origin xyz="-0.52 -0.4 0.43" rpy="0 0 0"/>
@@ -39,5 +39,5 @@
     <visual>
       <geometry>
-        <mesh filename="package://robot_description/meshes/base.dae"/>
+        <mesh filename="package://robot_a_description/meshes/base.dae"/>
       </geometry>
       <origin xyz="-0.52 -0.4 0.0" rpy="0 0 0"/>
@@ -45,5 +45,5 @@
     <collision>
       <geometry>
-        <mesh filename="package://robot_description/meshes/base.dae"/>
+        <mesh filename="package://robot_a_description/meshes/base.dae"/>
       </geometry>
       <origin xyz="-0.52 -0.4 0.0" rpy="0 0 0"/>
@@ -60,5 +60,5 @@
     </inertial>
   </link>
-  <xacro:include filename="$(find robot_description)/urdf/arm.xacro" />
+  <xacro:include filename="$(find robot_a_description)/urdf/arm.xacro" />
   <!-- Conectar la base del brazo (arm_base_link) a la segunda plataforma del robot (base_second_link) -->
   <joint name="arm_base_connection_joint" type="fixed">
@@ -77,5 +77,5 @@
     <visual>
       <geometry>
-        <mesh filename="package://robot_description/meshes/rasp.dae" scale="0.14 0.14 0.14"/>
+        <mesh filename="package://robot_a_description/meshes/rasp.dae" scale="0.14 0.14 0.14"/>
       </geometry>
       <origin xyz="0.9 -1.25 0" rpy="0 0 1.57"/>
@@ -83,5 +83,5 @@
     <collision>
       <geometry>
-        <mesh filename="package://robot_description/meshes/rasp.dae" scale="0.14 0.14 0.14"/>
+        <mesh filename="package://robot_a_description/meshes/rasp.dae" scale="0.14 0.14 0.14"/>
       </geometry>
       <origin xyz="0.9 -1.25 0" rpy="0 0 1.57"/>
@@ -103,5 +103,5 @@
     <visual>
       <geometry>
-        <mesh filename="package://robot_description/meshes/rasp.dae" scale="0.14 0.14 0.14"/>
+        <mesh filename="package://robot_a_description/meshes/rasp.dae" scale="0.14 0.14 0.14"/>
       </geometry>
       <origin xyz="0.9 -1.25 0" rpy="0 0 1.57"/>
@@ -109,5 +109,5 @@
     <collision>
       <geometry>
-        <mesh filename="package://robot_description/meshes/rasp.dae" scale="0.14 0.14 0.14"/>
+        <mesh filename="package://robot_a_description/meshes/rasp.dae" scale="0.14 0.14 0.14"/>
       </geometry>
       <origin xyz="0.9 -1.25 0" rpy="0 0 1.57"/>
@@ -205,5 +205,5 @@
     <visual>
       <geometry>
-        <mesh filename="package://robot_description/meshes/battery.dae" scale="13.0 6.0 6.0"/>
+        <mesh filename="package://robot_a_description/meshes/battery.dae" scale="13.0 6.0 6.0"/>
       </geometry>
       <origin xyz="0 4.5 0.05" rpy="1.57 0 1.57"/>
@@ -211,5 +211,5 @@
     <collision>
       <geometry>
-        <mesh filename="package://robot_description/meshes/battery.dae" scale="13.0 6.0 6.0"/>
+        <mesh filename="package://robot_a_description/meshes/battery.dae" scale="13.0 6.0 6.0"/>
       </geometry>
       <origin xyz="0 4.5 0.05" rpy="1.57 0 1.57"/>
@@ -292,5 +292,5 @@
         <!-- cylinder length="0.0206" radius="0.0550"/-->
         <!--cylinder length="0.20" radius="0.26"/-->
-        <mesh filename="package://robot_description/meshes/wheel.dae" scale="8.0 8.0 8.0"/>
+        <mesh filename="package://robot_a_description/meshes/wheel.dae" scale="8.0 8.0 8.0"/>
       </geometry>
       <origin rpy="0.0 0 0" xyz="0 0 0"/>
@@ -320,5 +320,5 @@
       <geometry>
   <!--cylinder length="0.20" radius="0.26"/-->
-        <mesh filename="package://robot_description/meshes/wheel.dae" scale="8.0 8.0 8.0"/>
+        <mesh filename="package://robot_a_description/meshes/wheel.dae" scale="8.0 8.0 8.0"/>
       </geometry>
       <origin rpy="0.0 0 0" xyz="0 0 0"/>
@@ -408,5 +408,5 @@
     <visual>
       <geometry>
-        <mesh filename="package://robot_description/meshes/camera.dae" scale="4.0 4.0 4.0"/>
+        <mesh filename="package://robot_a_description/meshes/camera.dae" scale="4.0 4.0 4.0"/>
       </geometry>
       <origin xyz="0.0 0 0" rpy="0 0 0"/>
@@ -414,5 +414,5 @@
     <collision>
       <geometry>
-        <mesh filename="package://robot_description/meshes/camera.dae" scale="4.0 4.0 4.0"/>
+        <mesh filename="package://robot_a_description/meshes/camera.dae" scale="4.0 4.0 4.0"/>
       </geometry>
       <origin xyz="0.0 0 0" rpy="0 0 0"/>

Commit message: update comments to english

File: src/machine/robot_a_description/urdf/arm.xacro (robot description, xacro)
@@ -1,13 +1,13 @@
 <?xml version="1.0"?>
 <robot xmlns:xacro="http://www.ros.org/wiki/xacro">
-  <!-- Incluir propiedades comunes para materiales (ya se incluye en robot.xacro, pero se añade para claridad) -->
+  <!-- Include common properties for materials (already included in robot.xacro, but added for clarity) -->
   <xacro:include filename="$(find robot_a_description)/urdf/common_properties.xacro" />
-  <!-- Base del brazo (se conectará a la base del robot principal) -->
+  <!-- Arm base (will connect to the main robot base) -->
   <link name="arm_base_link">
     <visual>
       <geometry>
-        <box size="0.15 0.15 0.03"/> <!-- Base más ancha y plana -->
+        <box size="0.15 0.15 0.03"/> <!-- Wider and flatter base -->
       </geometry>
-      <material name="grey"/> <!-- Usando material de common_properties -->
+      <material name="grey"/> <!-- Using material from common_properties -->
     </visual>
     <collision>
@@ -24,10 +24,10 @@
     </inertial>
   </link>
-  <!-- Articulación del hombro (revolute para rotación horizontal) -->
+  <!-- Shoulder joint (revolute for horizontal rotation) -->
   <joint name="shoulder_joint" type="revolute">
     <parent link="arm_base_link"/>
     <child link="shoulder_link"/>
-    <origin xyz="0 0 0.015" rpy="0 0 0"/> <!-- Posición encima de la base del brazo -->
-    <axis xyz="0 0 1"/> <!-- Rotación alrededor del eje Z (horizontal) -->
+    <origin xyz="0 0 0.015" rpy="0 0 0"/> <!-- Position above the arm base -->
+    <axis xyz="0 0 1"/> <!-- Rotation around the Z-axis (horizontal) -->
     <limit lower="-1.8" upper="1.8" effort="100" velocity="0.5"/>
   </joint>
@@ -35,8 +35,8 @@
     <visual>
       <geometry>
-        <cylinder radius="0.05" length="0.25"/> <!-- Cilindro para el segmento del brazo -->
+        <cylinder radius="0.05" length="0.25"/> <!-- Cylinder for the arm segment -->
       </geometry>
-      <origin xyz="0 0 0.125" rpy="0 0 0"/> <!-- Centrar el cilindro para que extienda hacia arriba -->
-      <material name="blue"/> <!-- Color diferente para el segmento -->
+      <origin xyz="0 0 0.125" rpy="0 0 0"/> <!-- Center the cylinder to extend upwards -->
+      <material name="blue"/> <!-- Different color for the segment -->
     </visual>
     <collision>
@@ -54,10 +54,10 @@
     </inertial>
   </link>
-  <!-- Articulación del codo (revolute para rotación vertical) -->
+  <!-- Elbow joint (revolute for vertical rotation) -->
   <joint name="elbow_joint" type="revolute">
     <parent link="shoulder_link"/>
     <child link="elbow_link"/>
-    <origin xyz="0 0 0.25" rpy="0 0 0"/> <!-- En la parte superior del eslabón del hombro -->
-    <axis xyz="0 1 0"/> <!-- Rotación alrededor del eje Y (vertical) -->
+    <origin xyz="0 0 0.25" rpy="0 0 0"/> <!-- At the top of the shoulder link -->
+    <axis xyz="0 1 0"/> <!-- Rotation around the Y-axis (vertical) -->
     <limit lower="-1.8" upper="1.8" effort="100" velocity="0.5"/>
   </joint>
@@ -65,5 +65,5 @@
     <visual>
       <geometry>
-        <cylinder radius="0.04" length="0.20"/> <!-- Cilindro más pequeño -->
+        <cylinder radius="0.04" length="0.20"/> <!-- Smaller cylinder -->
       </geometry>
       <origin xyz="0 0 0.1" rpy="0 0 0"/>
@@ -84,10 +84,10 @@
     </inertial>
   </link>
-  <!-- Articulación de la muñeca (revolute para rotación vertical) -->
+  <!-- Wrist joint (revolute for vertical rotation) -->
   <joint name="wrist_joint" type="revolute">
     <parent link="elbow_link"/>
     <child link="wrist_link"/>
-    <origin xyz="0 0 0.2" rpy="0 0 0"/> <!-- En la parte superior del eslabón del codo -->
-    <axis xyz="0 1 0"/> <!-- Rotación alrededor del eje Y (vertical) -->
+    <origin xyz="0 0 0.2" rpy="0 0 0"/> <!-- At the top of the elbow link -->
+    <axis xyz="0 1 0"/> <!-- Rotation around the Y-axis (vertical) -->
     <limit lower="-1.8" upper="1.8" effort="100" velocity="0.5"/>
   </joint>
@@ -95,5 +95,5 @@
     <visual>
       <geometry>
-        <cylinder radius="0.03" length="0.08"/> <!-- Cilindro aún más pequeño -->
+        <cylinder radius="0.03" length="0.08"/> <!-- Even smaller cylinder -->
       </geometry>
       <origin xyz="0 0 0.04" rpy="0 0 0"/>
@@ -114,14 +114,14 @@
     </inertial>
   </link>
-  <!-- Efector final (puede ser un simple cubo o un gripper más complejo) -->
+  <!-- End effector (can be a simple cube or a more complex gripper) -->
   <joint name="end_effector_joint" type="fixed">
     <parent link="wrist_link"/>
     <child link="end_effector_link"/>
-    <origin xyz="0 0 0.08" rpy="0 0 0"/> <!-- Posición al final de la muñeca -->
+    <origin xyz="0 0 0.08" rpy="0 0 0"/> <!-- Position at the end of the wrist -->
   </joint>
   <link name="end_effector_link">
     <visual>
       <geometry>
-        <box size="0.06 0.06 0.03"/> <!-- Caja simple para el efector final -->
+        <box size="0.06 0.06 0.03"/> <!-- Simple box for the end effector -->
       </geometry>
       <material name="grey"/>

File: src/machine/robot_b_description/urdf/robot.gazebo.xacro (robot description, xacro)
@@ -22,9 +22,9 @@
     </plugin>
   </gazebo>
-  <!-- Propiedades de Gazebo para las ruedas -->
-  <!-- Ruedas motrices (delanteras): alta fricción para tracción -->
+  <!-- Gazebo properties for the wheels -->
+  <!-- Driving wheels (front): high friction for traction -->
   <gazebo reference="front_left_wheel_link">
-    <kp>1000000.0</kp> <!-- Constante elástica de contacto -->
-    <kd>100.0</kd> <!-- Constante de amortiguación de contacto -->
+    <kp>1000000.0</kp> <!-- Contact stiffness constant -->
+    <kd>100.0</kd> <!-- Contact damping constant -->
     <minDepth>0.001</minDepth>
     <maxVel>1.0</maxVel>
@@ -36,5 +36,5 @@
     <maxVel>1.0</maxVel>
   </gazebo>
-  <!-- Ruedas pasivas (traseras): muy baja fricción para permitir el deslizamiento lateral durante el giro -->
+  <!-- Passive wheels (rear): very low friction to allow lateral slip during turning -->
   <gazebo reference="back_left_wheel_link">
     <kp>1000000.0</kp>

File: src/machine/robot_b_description/urdf/robot.xacro (robot description, xacro)
@@ -5,7 +5,7 @@
   <!-- Gazebo configuration -->
   <xacro:include filename="$(find robot_b_description)/urdf/robot.gazebo.xacro" />
-  <!-- Link base_footprint (convención ROS para la base del robot) -->
+  <!-- Link base_footprint (ROS convention for the robot's base) -->
   <link name="base_footprint"/>
-  <!-- Joint que conecta base_footprint con base_link -->
+  <!-- Joint connecting base_footprint to base_link -->
   <joint name="base_joint" type="fixed">
     <origin xyz="0 0 0.2" rpy="0 0 0" />
@@ -13,9 +13,9 @@
     <child link="base_link" />
   </joint>
-  <!-- Link principal del robot (cuerpo central) -->
+  <!-- Main link of the robot (central body) -->
   <link name="base_link">
     <visual>
       <geometry>
-        <box size="0.6 0.4 0.2"/> <!-- Un cubo simple para la base -->
+        <box size="0.6 0.4 0.2"/> <!-- A simple box for the base -->
       </geometry>
       <material name="grey"/>
@@ -28,6 +28,6 @@
     <inertial>
       <origin xyz="0 0 0"/>
-      <mass value="10.0"/> <!-- Masa de la base -->
-      <!-- Momentos de inercia para un cubo -->
+      <mass value="10.0"/> <!-- Base mass -->
+      <!-- Inertia moments for a box -->
       <inertia ixx="1.0" ixy="0.0" ixz="0.0"
                iyy="1.0" iyz="0.0"
@@ -35,17 +35,17 @@
     </inertial>
   </link>
-  <!-- Macro para definir una rueda, facilitando la creación de las cuatro -->
+  <!-- Macro to define a wheel, facilitating the creation of all four -->
   <xacro:macro name="wheel" params="prefix parent_link x_offset y_offset z_offset">
     <joint name="${prefix}_wheel_joint" type="continuous">
       <parent link="${parent_link}"/>
       <child link="${prefix}_wheel_link"/>
-      <!-- rpy="-1.570795 0 0" rota la rueda para que el eje Z apunte hacia afuera (horizontal) -->
+      <!-- rpy="-1.570795 0 0" rotates the wheel so that the Z-axis points outward (horizontal) -->
       <origin xyz="${x_offset} ${y_offset} ${z_offset} " rpy="-1.570795 0 0"/>
-      <axis xyz="0 0 1"/> <!-- El eje de rotación de la rueda es su propio eje Z local -->
+      <axis xyz="0 0 1"/> <!-- The wheel's rotation axis is its own local Z-axis -->
     </joint>
     <link name="${prefix}_wheel_link">
       <visual>
         <geometry>
-          <cylinder radius="0.1" length="0.05"/> <!-- Un cilindro para la rueda -->
+          <cylinder radius="0.1" length="0.05"/> <!-- A cylinder for the wheel -->
         </geometry>
         <material name="black"/>
@@ -58,6 +58,6 @@
       <inertial>
         <origin xyz="0 0 0"/>
-        <mass value="0.5"/> <!-- Masa de la rueda -->
-        <!-- Momentos de inercia para un cilindro -->
+        <mass value="0.5"/> <!-- Wheel mass -->
+        <!-- Inertia moments for a cylinder -->
         <inertia ixx="0.002" ixy="0.0" ixz="0.0"
                  iyy="0.002" iyz="0.0"
@@ -66,12 +66,12 @@
     </link>
   </xacro:macro>
-  <!-- Instanciamos las cuatro ruedas usando la macro -->
-  <!-- Rueda Delantera Izquierda -->
+  <!-- Instantiate the four wheels using the macro -->
+  <!-- Front Left Wheel -->
   <xacro:wheel prefix="front_left" parent_link="base_link" x_offset="0.2" y_offset="0.225" z_offset="-0.1"/>
-  <!-- Rueda Delantera Derecha -->
+  <!-- Front Right Wheel -->
   <xacro:wheel prefix="front_right" parent_link="base_link" x_offset="0.2" y_offset="-0.225" z_offset="-0.1"/>
-  <!-- Rueda Trasera Izquierda -->
+  <!-- Back Left Wheel -->
   <xacro:wheel prefix="back_left" parent_link="base_link" x_offset="-0.2" y_offset="0.225" z_offset="-0.1"/>
-  <!-- Rueda Trasera Derecha -->
+  <!-- Back Right Wheel -->
   <xacro:wheel prefix="back_right" parent_link="base_link" x_offset="-0.2" y_offset="-0.225" z_offset="-0.1"/>
 </robot>
